Commit message: Actualizo carpeta de ROS2 con últimos cambios

File: urdf/peperURDF.urdf (robot description, URDF)
Before this commit: robot peper, 12 links, 11 joints
Links:
- link l_sho: geometry collision mesh filename=package://rosPackage/urdf/peperParts/parts/copi_l_sho.stl scale=1 1 1; visual mesh filename=package://rosPackage/urdf/peperParts/parts/copi_l_sho.stl scale=1 1 1
- link r_sho: geometry collision mesh filename=package://rosPackage/urdf/peperParts/parts/copi_r_sho.stl scale=1 1 1; visual mesh filename=package://rosPackage/urdf/peperParts/parts/copi_r_sho.stl scale=1 1 1
Joints:
- joint base_to_legs: limit lower=-0.2 upper=0.3 effort=1000.0 velocity=0.5 -> lower=-0.3 upper=0.3 effort=1000.0 velocity=0.5
- joint chest_to_leg: limit lower=-0.2 upper=0.3 effort=1000.0 velocity=0.5 -> lower=-0.3 upper=0.6 effort=1000.0 velocity=0.5
- joint l_arm_to_shoulder: origin xyz=-0.039037 -0.001973 -0.190042 -> xyz=-0.002364 -0.002364 -0.190042
- joint l_sho_to_chest: limit lower=0 upper=2.09 effort=1000 velocity=0.5 -> lower=0 upper=1.57 effort=1000 velocity=0.5; origin xyz=-0.144 0.046 0.24  -> xyz=-0.19 0.046 0.24 
- joint r_arm_to_shoulder: origin xyz=0.039037 -0.001973 -0.190042 -> xyz=-0.002364 -0.002364 -0.190042
- joint r_sho_to_chest: limit lower=0 upper=-2.09 effort=1000.0 velocity=0.5 -> lower=0 upper=-1.57 effort=1000.0 velocity=0.5; origin xyz=0.144 0.046 0.24  -> xyz=0.19 0.046 0.24 

Commit message: fix: rotational and origin problems fixed and arms pitch added

File: urdf/peperURDF.urdf (robot description, URDF)
Before this commit: robot peper, 12 links, 11 joints
Links:
- added link l_sho_to_arm_intermediate
- added link l_sho_to_chest_intermediate
- added link r_sho_to_arm_intermediate
- added link r_sho_to_chest_intermediate
- link l_arm: geometry collision mesh filename=package://rosPackage/urdf/peperParts/parts/left_arm.stl scale=1 1 1; visual mesh filename=package://rosPackage/urdf/peperParts/parts/left_arm.stl scale=1 1 1
- link l_hand: geometry collision mesh filename=package://rosPackage/urdf/peperParts/parts/left_hand.stl scale=1 1 1; visual mesh filename=package://rosPackage/urdf/peperParts/parts/left_hand.stl scale=1 1 1
- link l_sho: geometry collision mesh filename=package://rosPackage/urdf/peperParts/parts/copi_left_sho.stl scale=1 1 1; visual mesh filename=package://rosPackage/urdf/peperParts/parts/copi_left_sho.stl scale=1 1 1
- link r_arm: geometry collision mesh filename=package://rosPackage/urdf/peperParts/parts/right_arm.stl scale=1 1 1; visual mesh filename=package://rosPackage/urdf/peperParts/parts/right_arm.stl scale=1 1 1
- link r_hand: geometry collision mesh filename=package://rosPackage/urdf/peperParts/parts/right_hand.stl scale=1 1 1; visual mesh filename=package://rosPackage/urdf/peperParts/parts/right_hand.stl scale=1 1 1
- link r_sho: geometry collision mesh filename=package://rosPackage/urdf/peperParts/parts/copi_right_sho.s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 scale=1 1 1; visual mesh filename=package://rosPackage/urdf/peperParts/parts/copi_right_sho.s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 scale=1 1 1
Joints:
- removed joint l_arm_to_shoulder
- removed joint l_sho_to_chest
- removed joint r_arm_to_shoulder
- removed joint r_sho_to_chest
- added joint l_arm_to_shoulder_pitch: type revolute, parent l_sho, child l_sho_to_arm_intermediate, origin xyz=-0.002364 -0.002364 -0.190042 rpy=0 0 0, axis 1 0 0, limit lower=-1.57 upper=0 effort=1000.0 velocity=0.5
- added joint l_arm_to_shoulder_yaw: type revolute, parent l_sho_to_arm_intermediate, child l_arm, origin xyz=0 0 0 rpy=0 0 0, axis 0 0 1, limit lower=-3.925 upper=0 effort=1000.0 velocity=0.5
- added joint l_sho_to_chest_pitch: type revolute, parent l_sho_to_chest_intermediate, child l_sho, origin xyz=0 0 0 rpy=0 0 0, axis 1 0 0, limit lower=-3.14 upper=0.785 effort=1000 velocity=0.5
- added joint l_sho_to_chest_roll: type revolute, parent chest, child l_sho_to_chest_intermediate, origin xyz=0.19 0.046 0.24 , axis 0 1 0, limit lower=-1.57 upper=0 effort=1000.0 velocity=0.5
- added joint r_arm_to_shoulder_pitch: type revolute, parent r_sho, child r_sho_to_arm_intermediate, origin xyz=-0.002364 -0.002364 -0.190042 rpy=0 0 0, axis 1 0 0, limit lower=-1.57 upper=0 effort=1000.0 velocity=0.5
- added joint r_arm_to_shoulder_yaw: type revolute, parent r_sho_to_arm_intermediate, child r_arm, origin xyz=0 0 0 rpy=0 0 0, axis 0 0 1, limit lower=0 upper=3.925 effort=1000.0 velocity=0.5
- added joint r_sho_to_chest_pitch: type revolute, parent r_sho_to_chest_intermediate, child r_sho, origin xyz=0 0 0 rpy=0 0 0, axis 1 0 0, limit lower=-3.14 upper=0.785 effort=1000 velocity=0.5
- added joint r_sho_to_chest_roll: type revolute, parent chest, child r_sho_to_chest_intermediate, origin xyz=-0.19 0.046 0.24 , axis 0 1 0, limit lower=0 upper=1.57 effort=1000 velocity=0.5
- joint base_to_legs: limit lower=-0.3 upper=0.3 effort=1000.0 velocity=0.5 -> lower=-0.6 upper=0.6 effort=1000.0 velocity=0.5
- joint l_hand_to_arm: origin xyz=0.001051 -0.006148 -0.169538 -> xyz=-0.001051 -0.006148 -0.169538
- joint r_hand_to_arm: origin xyz=-0.001051 -0.006148 -0.169538 -> xyz=0.001051 -0.006148 -0.169538

Commit message: feat: colitions in gazebo added

File: urdf/peperURDF.urdf (robot description, URDF)
Before this commit: robot peper, 16 links, 15 joints
Links:
- link base: mass None -> 15.485
- link base_link: mass None -> 0.1
- link chest: mass None -> 3.9953
- link head: mass None -> 1.5189
- link l_arm: mass None -> 0.16579
- link l_hand: mass None -> 0.27555
- link l_sho: mass None -> 0.50527
- link l_sho_to_arm_intermediate: mass None -> 0.27495
- link l_sho_to_chest_intermediate: mass None -> 0.3125
- link legs: mass None -> 3.4826
- link neck: mass None -> 0.27391
- link r_arm: mass None -> 0.16579
- link r_hand: mass None -> 0.27555
- link r_sho: mass None -> 0.50527
- link r_sho_to_arm_intermediate: mass None -> 0.27495
- link r_sho_to_chest_intermediate: mass None -> 0.3125
Joints:
- joint base_to_base: origin xyz=0 0 0 rpy= 0 0 0 -> xyz=0 0 0 rpy=0 0 0
- joint base_to_legs: axis 1.0 0 0 -> 1 0 0; limit lower=-0.6 upper=0.6 effort=1000.0 velocity=0.5 -> lower=-0.6 upper=0.6 effort=1000 velocity=0.5
- joint chest_to_leg: axis 1.0 0 0 -> 1 0 0; limit lower=-0.3 upper=0.6 effort=1000.0 velocity=0.5 -> lower=-0.3 upper=0.6 effort=1000 velocity=0.5; origin xyz=0 0 0.325  -> xyz=0 0 0.325
- joint head_to_chest: limit lower=-0.523 upper=0.785 effort=1000.0 velocity=0.5 -> lower=-0.523 upper=0.785 effort=1000 velocity=0.5; origin xyz=0 0 0.03  -> xyz=0 0 0.03
- joint l_arm_to_shoulder_pitch: limit lower=-1.57 upper=0 effort=1000.0 velocity=0.5 -> lower=-1.57 upper=0 effort=1000 velocity=0.5; origin xyz=-0.002364 -0.002364 -0.190042 rpy=0 0 0 -> xyz=-0.002364 -0.002364 -0.190042
- joint l_arm_to_shoulder_yaw: limit lower=-3.925 upper=0 effort=1000.0 velocity=0.5 -> lower=-3.925 upper=0 effort=1000 velocity=0.5; origin xyz=0 0 0 rpy=0 0 0 -> xyz=0 0 0
- joint l_sho_to_chest_pitch: origin xyz=0 0 0 rpy=0 0 0 -> xyz=0 0 0
- joint l_sho_to_chest_roll: limit lower=-1.57 upper=0 effort=1000.0 velocity=0.5 -> lower=-1.57 upper=0 effort=1000 velocity=0.5; origin xyz=0.19 0.046 0.24  -> xyz=0.19 0.046 0.24
- joint neck_to_chest: limit lower=-0.75 upper=0.75 effort=1000.0 velocity=0.5 -> lower=-0.75 upper=0.75 effort=1000 velocity=0.5
- joint r_arm_to_shoulder_pitch: limit lower=-1.57 upper=0 effort=1000.0 velocity=0.5 -> lower=-1.57 upper=0 effort=1000 velocity=0.5; origin xyz=-0.002364 -0.002364 -0.190042 rpy=0 0 0 -> xyz=-0.002364 -0.002364 -0.190042
- joint r_arm_to_shoulder_yaw: limit lower=0 upper=3.925 effort=1000.0 velocity=0.5 -> lower=0 upper=3.925 effort=1000 velocity=0.5; origin xyz=0 0 0 rpy=0 0 0 -> xyz=0 0 0
- joint r_sho_to_chest_pitch: origin xyz=0 0 0 rpy=0 0 0 -> xyz=0 0 0
- joint r_sho_to_chest_roll: origin xyz=-0.19 0.046 0.24  -> xyz=-0.19 0.046 0.24
